Commit message: Rename all x2 identifiers to ff_master across the repo.
Rename model files, demo script, MJCF classes, and documentation strings while keeping the assets/ff-master directory path.

Co-authored-by: Cursor <cursoragent@cursor.com>

File: assets/ff-master/ff_master_fist.urdf (robot description, URDF)
Before this commit: robot x2t2.5, 41 links, 40 joints
Links:
- removed link base_link
- removed link left_wrist_pitch_link
- removed link left_wrist_roll_link
- removed link lidar_chest_front
- removed link rgb_head_center
- removed link rgb_head_rear
- removed link rgbd_head_front
- removed link right_wrist_pitch_link
- removed link right_wrist_roll_link
- removed link stereo_head_front
- added link rgb_head_center_link, mass 0.00725056310822806; visual mesh filename=./meshes/rgb_head_center_link.STL
- added link rgb_head_rear_link, mass 0.00293607901610696; visual mesh filename=./meshes/rgb_head_rear_link.STL
- added link rgbd_head_front_link, mass 0.00266754316393765; visual mesh filename=./meshes/rgbd_head_front_link.STL
- added link stereo_head_front_link, mass 0.032843906465572; visual mesh filename=./meshes/stereo_head_front_link.STL
- link imu_in_head_link: mass None -> 0.00969276520032405
- link left_wrist_yaw_link: mass 0.360708 -> 0.767123; geometry collision mesh filename=./meshes/left_wrist_fist_link.STL; visual mesh filename=./meshes/left_wrist_fist_link.STL
- link right_wrist_yaw_link: mass 0.372787 -> 0.767125; geometry collision mesh filename=./meshes/right_wrist_fist_link.STL; visual mesh filename=./meshes/right_wrist_fist_link.STL
- link torso_link: mass 10.144138 -> 9.464653
Joints:
- removed joint base_link_joint
- removed joint left_wrist_pitch_joint
- removed joint left_wrist_roll_joint
- removed joint lidar_chest_front
- removed joint rgb_head_center
- removed joint rgb_head_rear
- removed joint rgbd_head_front
- removed joint right_wrist_pitch_joint
- removed joint right_wrist_roll_joint
- removed joint stereo_head_front
- added joint rgb_head_center_joint: type fixed, parent head_pitch_link, child rgb_head_center_link, origin xyz=0.0683999822649913 -0.000217129490632628 0.0499999897221556 rpy=-1.57079647705046 0 -1.57397317220857, axis 0 0 0
- added joint rgb_head_rear_joint: type fixed, parent head_pitch_link, child rgb_head_rear_link, origin xyz=-0.0833995753645274 0.000264949140505621 0 rpy=-1.57079617653953 0 1.56761942309941, axis 0 0 0
- added joint rgbd_head_front_joint: type fixed, parent head_pitch_link, child rgbd_head_front_link, origin xyz=0.057609600436012 -0.0111832348707392 -0.0483697394600023 rpy=2.26893066700097 0 1.5707963267949, axis 0 0 0
- added joint stereo_head_front_joint: type fixed, parent head_pitch_link, child stereo_head_front_link, origin xyz=0.0679950106115899 0.0297843084328545 0.0499998893534674 rpy=-1.57079647705046 0 -1.57397317220857, axis 0 0 0
- joint head_pitch_joint: origin xyz=0 0 0.0889 rpy=0 0 0 -> xyz=0 0 0.0888999999995007 rpy=0 0 0
- joint left_wrist_yaw_joint: axis 0 0 1 -> 0 0 -1; origin xyz=-0.0132797235062217 -9.75487744990788E-05 -0.120575783591803 rpy=0 0 0 -> xyz=-0.01328 -9.7549E-05 -0.12058 rpy=0 0 0

File: assets/ff-master/ff_master_ultra.urdf (robot description, URDF)
Before this commit: robot x2_t2.5, 35 links, 34 joints
Links:
- removed link rgb_head_center_link
- removed link rgb_head_rear_link
- removed link rgbd_head_front_link
- removed link stereo_head_front_link
- added link base_link
- added link left_wrist_pitch_link, mass 0.292062; collision mesh filename=./meshes/left_wrist_pitch_link.STL; visual mesh filename=./meshes/left_wrist_pitch_link.STL
- added link left_wrist_roll_link, mass 0.30304; collision mesh filename=./meshes/left_wrist_roll_link.STL; visual mesh filename=./meshes/left_wrist_roll_link.STL
- added link lidar_chest_front
- added link rgb_head_center; visual mesh filename=./meshes/rgb_head_center_link.STL
- added link rgb_head_rear; visual mesh filename=./meshes/rgb_head_rear_link.STL
- added link rgbd_head_front; visual mesh filename=./meshes/rgbd_head_front_link.STL
- added link right_wrist_pitch_link, mass 0.279175; collision mesh filename=./meshes/right_wrist_pitch_link.STL; visual mesh filename=./meshes/right_wrist_pitch_link.STL
- added link right_wrist_roll_link, mass 0.303847; collision mesh filename=./meshes/right_wrist_roll_link.STL; visual mesh filename=./meshes/right_wrist_roll_link.STL
- added link stereo_head_front; visual mesh filename=./meshes/stereo_head_front_link.STL
- link imu_in_head_link: mass 0.00969276520032405 -> None
- link left_wrist_yaw_link: mass 0.767123 -> 0.360708; geometry collision mesh filename=./meshes/left_wrist_yaw_link.STL; visual mesh filename=./meshes/left_wrist_yaw_link.STL
- link right_wrist_yaw_link: mass 0.767125 -> 0.372787; geometry collision mesh filename=./meshes/right_wrist_yaw_link.STL; visual mesh filename=./meshes/right_wrist_yaw_link.STL
- link torso_link: mass 9.464653 -> 10.144138
Joints:
- removed joint rgb_head_center_joint
- removed joint rgb_head_rear_joint
- removed joint rgbd_head_front_joint
- removed joint stereo_head_front_joint
- added joint base_link_joint: type fixed, parent base_link, child pelvis, origin xyz=0.0 0 0.0 rpy=0 0 0
- added joint left_wrist_pitch_joint: type revolute, parent left_wrist_yaw_link, child left_wrist_pitch_link, origin xyz=0.000490001227040848 0 -0.0819985359552045 rpy=0 -0.00597566028430406 0, axis 0 1 0, limit lower=-0.558 upper=0.558 effort=4.8 velocity=4.188
- added joint left_wrist_roll_joint: type revolute, parent left_wrist_pitch_link, child left_wrist_roll_link, origin xyz=0 0 0 rpy=0 0 0, axis 1 0 0, limit lower=-1.571 upper=0.724 effort=4.8 velocity=4.188
- added joint lidar_chest_front: type fixed, parent torso_link, child lidar_chest_front, origin xyz=0.102632855873251 0 0.181586916322065 rpy=-1.5707963267949 0 0, axis 0 0 0
- added joint rgb_head_center: type fixed, parent head_pitch_link, child rgb_head_center, origin xyz=0.0684 -0.00021713 0.05 rpy=-1.5708 0 -1.574, axis 0 0 0
- added joint rgb_head_rear: type fixed, parent head_pitch_link, child rgb_head_rear, origin xyz=-0.0834 0.00026495 0 rpy=-1.5708 0 1.5676, axis 0 0 0
- added joint rgbd_head_front: type fixed, parent head_pitch_link, child rgbd_head_front, origin xyz=0.05761 -0.011183 -0.04837 rpy=2.2689 0 1.5708, axis 0 0 0
- added joint right_wrist_pitch_joint: type revolute, parent right_wrist_yaw_link, child right_wrist_pitch_link, origin xyz=0 0 -0.081799999999999 rpy=0 0 -3.27341932546355E-05, axis 0 1 0, limit lower=-0.558 upper=0.558 effort=4.8 velocity=4.188
- added joint right_wrist_roll_joint: type revolute, parent right_wrist_pitch_link, child right_wrist_roll_link, origin xyz=0 0 0 rpy=0 0 0, axis 1 0 0, limit lower=-0.724 upper=1.571 effort=4.8 velocity=4.188
- added joint stereo_head_front: type fixed, parent head_pitch_link, child stereo_head_front, origin xyz=0.067995 0.029784 0.05 rpy=-1.5708 0 -1.574, axis 0 0 0
- joint head_pitch_joint: origin xyz=0 0 0.0888999999995007 rpy=0 0 0 -> xyz=0 0 0.0889 rpy=0 0 0
- joint left_wrist_yaw_joint: axis 0 0 -1 -> 0 0 1; origin xyz=-0.01328 -9.7549E-05 -0.12058 rpy=0 0 0 -> xyz=-0.0132797235062217 -9.75487744990788E-05 -0.120575783591803 rpy=0 0 0
